Commit message: Error loading moveit model, saving changes so that reverts can be made

File: ws_AF/src/baxter_common/baxter_description/urdf/baxter_base/baxter_base.urdf.xacro (robot description, xacro)
@@ -512,5 +512,4 @@
     <child link="right_arm_mount"/>
   </joint>
-  <!--
   <joint name="right_s0" type="revolute">
     <origin rpy="0 0 0" xyz="0.055695 0 0.011038"/>
@@ -586,5 +585,5 @@
     <limit effort="15.0" lower="-3.059" upper="3.059" velocity="4.0"/>
     <dynamics damping="0.7" friction="0.0"/>
-  </joint> -->
+  </joint>
   <joint name="right_hand" type="fixed">
     <origin rpy="0 0 0" xyz="0 0 0.11355"/>
@@ -881,5 +880,4 @@
     <child link="left_arm_mount"/>
   </joint>
-  <!--
   <joint name="left_s0" type="revolute">
     <origin rpy="0 0 0" xyz="0.055695 0 0.011038"/>
@@ -955,5 +953,5 @@
     <limit effort="15.0" lower="-3.059" upper="3.059" velocity="4.0"/>
     <dynamics damping="0.7" friction="0.0"/>
-  </joint> -->
+  </joint>
   <joint name="left_hand" type="fixed">
     <origin rpy="0 0 0" xyz="0 0 0.11355"/>

File: ws_AF/src/baxter_common/baxter_description/urdf/left_end_effector.urdf.xacro (robot description, xacro)
@@ -2,18 +2,5 @@
 <robot name="left_end_effector" xmlns:xacro="http://www.ros.org/wiki/xacro">
   <!-- Include the Robotiq 2F-85 gripper Xacro file -->
-  <!-- <xacro:include filename="$(find rethink_ee_description)/urdf/electric_gripper/rethink_electric_gripper.xacro" /> -->
-  <xacro:include filename="$(find robotiq_2f_85_gripper_visualization)/urdf/robotiq_arg2f_85_model_macro.xacro" />
-  <!-- <xacro:rethink_electric_gripper side="left"
-                                  l_finger="extended_narrow"
-                                  l_finger_slot="2"
-                                  l_finger_tip="paddle_tip"
-                                  l_finger_grasp="inner"
-                                  r_finger="extended_narrow"
-                                  r_finger_slot="2"
-                                  r_finger_tip="paddle_tip"
-                                  r_finger_grasp="inner"/> -->
-  <!-- Define the Robotiq 2F-85 gripper components -->
-  <xacro:robotiq_arg2f_base_link prefix="left_" />
-  <xacro:finger_links prefix="left_" fingerprefix="left_finger" stroke="0.085" />
-  <xacro:finger_joints prefix="left_" fingerprefix="left_finger" reflect="0" />
+  <xacro:include filename="$(find robotiq_2f_85_gripper_vis)/urdf/robotiq_arg2f_85_model_macro.xacro" />
+  <xacro:left_gripper prefix="" /> <!-- loads the model in -->
 </robot>

File: ws_AF/src/moveit_robots/baxter_moveit_config/baxter_moveit_config/config/baxter.srdf.xacro (robot description, xacro)
@@ -1,27 +1,28 @@
 <?xml version="1.0" ?>
 <robot name="baxter" xmlns:xacro="http://www.ros.org/wiki/xacro">
-  <!-- Arguments -->
+  <!-- Arguments (go into baxter_base)-->
   <xacro:arg name="left_tip_name" default="left_gripper"/>
   <xacro:arg name="right_tip_name" default="right_gripper"/>
-  <xacro:arg name="left_electric_gripper" default="false"/>
-  <xacro:arg name="right_electric_gripper" default="false"/>
-  <xacro:arg name="left_robotiq_gripper" default="false"/>
+  <!--<xacro:arg name="left_robotiq_gripper" default="false"/> -->
   <!-- Base Configuration -->
   <xacro:include filename="$(find baxter_moveit_config)/config/baxter_base.srdf.xacro" />
   <xacro:baxter_base left_tip_name="$(arg left_tip_name)" right_tip_name="$(arg right_tip_name)"/>
   <!--Left End Effector Collisions-->
-  <!--<xacro:include filename="$(find baxter_moveit_config)/config/default_gripper.srdf.xacro" />
-  <xacro:default_gripper side="left"/>
-  <xacro:if value="$(arg left_electric_gripper)">
+  <xacro:include filename="$(find baxter_moveit_config)/config/left_default_gripper.srdf.xacro" />
+  <xacro:left_default_gripper side="left"/>
+  <xacro:arg name="left_electric_gripper" default="false"/>
+  <!-- <xacro:if value="$(arg left_electric_gripper)">
     <xacro:include filename="$(find baxter_moveit_config)/config/rethink_electric_gripper.srdf.xacro" />
     <xacro:rethink_electric_gripper side="left"/>
   </xacro:if> -->
-  <xacro:if value="$(arg left_robotiq_gripper)"> <!-- Conditional inclusion of Robotiq gripper -->
-    <xacro:include filename="$(find robotiq_2f_85_gripper_visualization)/urdf/robotiq_arg2f_85_model_macro.xacro" /> <!-- Replace with actual path -->
-    <xacro:robotiq_arg2f_85_model_macro side="left"/>
+  <!-- Conditional inclusion of Robotiq gripper -->
+  <xacro:if value="$(arg left_electric_gripper)">
+    <xacro:include filename="$(find baxter_moveit_config)/config/robotiq_gripper.srdf.xacro" />
+    <xacro:robotiq_gripper side="left"/>
   </xacro:if>
   <!--Right End Effector Collisions-->
   <xacro:include filename="$(find baxter_moveit_config)/config/default_gripper.srdf.xacro" />
   <xacro:default_gripper side="right"/>
+  <xacro:arg name="right_electric_gripper" default="false"/>
   <xacro:if value="$(arg right_electric_gripper)">
     <xacro:include filename="$(find baxter_moveit_config)/config/rethink_electric_gripper.srdf.xacro" />

File: ws_AF/src/moveit_robots/baxter_moveit_config/baxter_moveit_config/config/rethink_electric_gripper.srdf.xacro (robot description, xacro)
@@ -16,7 +16,14 @@
     <disable_collisions link1="${side}_gripper" link2="${gripper_side}_gripper_r_finger" reason="Default" />
     <disable_collisions link1="${side}_gripper" link2="${gripper_side}_gripper_r_finger_tip" reason="Never" />
-    <disable_collisions link1="${gripper_side}_gripper_l_finger" link2="${gripper_side}_gripper_l_finger_tip" reason="Adjacent" />
+    <!-- Between links -->
+    <disable_collisions link1="${gripper_side}_gripper_l_finger" link2="${gripper_side}_gripper_r_finger_tip" reason="Adjacent" />
     <disable_collisions link1="${gripper_side}_gripper_l_finger" link2="${gripper_side}_gripper_r_finger" reason="Never" />
     <disable_collisions link1="${gripper_side}_gripper_l_finger" link2="${gripper_side}_gripper_r_finger_tip" reason="Never" />
+    <disable_collisions link1="${gripper_side}_gripper_l_finger_tip" link2="${gripper_side}_gripper_r_finger" reason="Never" />
+    <disable_collisions link1="${gripper_side}_gripper_r_finger" link2="${gripper_side}_gripper_r_finger_tip" reason="Adjacent" />
+    <disable_collisions link1="${gripper_side}_gripper_l_finger_tip" link2="${gripper_side}_gripper_r_finger_tip" reason="Never" />
+    <disable_collisions link1="${gripper_side}_gripper_l_finger" link2="${gripper_side}_gripper_l_finger_tip" reason="Never" />
+    <disable_collisions link1="${gripper_side}_gripper_r_finger" link2="${gripper_side}_gripper_r_finger_tip" reason="Never" />
+    <!-- l -->
     <disable_collisions link1="${gripper_side}_gripper_l_finger" link2="${side}_hand" reason="Never" />
     <disable_collisions link1="${gripper_side}_gripper_l_finger" link2="${side}_hand_accelerometer" reason="Never" />
@@ -28,5 +35,4 @@
     <disable_collisions link1="${gripper_side}_gripper_l_finger" link2="${side}_upper_forearm_visual" reason="Never" />
     <disable_collisions link1="${gripper_side}_gripper_l_finger" link2="${side}_wrist" reason="Never" />
-    <disable_collisions link1="${gripper_side}_gripper_l_finger_tip" link2="${gripper_side}_gripper_r_finger" reason="Never" />
     <disable_collisions link1="${gripper_side}_gripper_l_finger_tip" link2="${side}_hand" reason="Never" />
     <disable_collisions link1="${gripper_side}_gripper_l_finger_tip" link2="${side}_hand_accelerometer" reason="Never" />
@@ -39,5 +45,5 @@
     <disable_collisions link1="${gripper_side}_gripper_l_finger_tip" link2="${side}_upper_forearm_visual" reason="Never" />
     <disable_collisions link1="${gripper_side}_gripper_l_finger_tip" link2="${side}_wrist" reason="Never" />
-    <disable_collisions link1="${gripper_side}_gripper_r_finger" link2="${gripper_side}_gripper_r_finger_tip" reason="Adjacent" />
+    <!-- r -->
     <disable_collisions link1="${gripper_side}_gripper_r_finger" link2="${side}_hand" reason="Never" />
     <disable_collisions link1="${gripper_side}_gripper_r_finger" link2="${side}_hand_accelerometer" reason="Never" />
@@ -59,24 +65,4 @@
     <disable_collisions link1="${gripper_side}_gripper_r_finger_tip" link2="${side}_upper_forearm_visual" reason="Never" />
     <disable_collisions link1="${gripper_side}_gripper_r_finger_tip" link2="${side}_wrist" reason="Never" />
-    <disable_collisions link1="${gripper_side}_gripper_l_finger_tip" link2="${gripper_side}_gripper_r_finger_tip" reason="Never" />
-    <disable_collisions link1="${gripper_side}_gripper_l_finger" link2="${gripper_side}_gripper_l_finger_tip" reason="Never" />
-    <disable_collisions link1="${gripper_side}_gripper_r_finger" link2="${gripper_side}_gripper_r_finger_tip" reason="Never" />
     </xacro:macro>
-    <!-- New Macro for Robotiq 2-Finger Gripper (Left) -->
-    <xacro:macro name="robotiq_2f_gripper" params="side">
-        <xacro:property name="gripper_side" value="${side[0]}" scope="local"/>
-        <!-- Add specific disable_collisions for the Robotiq 2F-85 Gripper -->
-        <disable_collisions link1="${side}_gripper_base" link2="${gripper_side}_gripper_finger_1" reason="Adjacent" />
-        <disable_collisions link1="${side}_gripper_base" link2="${gripper_side}_gripper_finger_2" reason="Adjacent" />
-        <disable_collisions link1="${side}_gripper_finger_1" link2="${gripper_side}_gripper_finger_2" reason="Adjacent" />
-        <disable_collisions link1="${gripper_side}_gripper_finger_1" link2="${side}_hand" reason="Never" />
-        <disable_collisions link1="${gripper_side}_gripper_finger_2" link2="${side}_hand" reason="Never" />
-        <!-- Add more disable_collisions as needed based on the robot's configuration -->
-    </xacro:macro>
-    <!-- Delete the below if it gives errors -->
-    <xacro:if value="$(arg left_gripper_is_robotiq)">
-        <xacro:robotiq_2f_gripper side="left"/>
-    </xacro:if>
-    <!-- Keep the original macro for the right side (if needed) -->
-    <xacro:rethink_electric_gripper side="right"/>
 </robot>
