Commit message: Reverting back to old moveit config and now loads moveit

File: setup/Backup/baxter_moveit_config/config/baxter.srdf.xacro (robot description, xacro)
@@ -9,4 +9,6 @@
   <xacro:baxter_base left_tip_name="$(arg left_tip_name)" right_tip_name="$(arg right_tip_name)"/>
   <!--Left End Effector Collisions-->
+  <!-- <xacro:include filename="$(find baxter_moveit_config)/config/left_default_gripper.srdf.xacro" />  REVERT 2-->
+  <!-- <xacro:left_default_gripper side="left"/> REVERT 2-->
   <xacro:include filename="$(find baxter_moveit_config)/config/default_gripper.srdf.xacro" />
   <xacro:default_gripper side="left"/>
@@ -18,6 +20,9 @@
   <!-- Conditional inclusion of Robotiq gripper -->
   <xacro:if value="$(arg left_electric_gripper)">
-    <xacro:include filename="$(find robotiq_2f_85_gripper_vis)/urdf/robotiq_gripper.srdf.xacro" />
+    <xacro:include filename="$(find baxter_moveit_config)/config/rethink_electric_gripper.srdf.xacro" />
+    <xacro:rethink_electric_gripper side="left"/>
+    <!--<xacro:include filename="$(find baxter_moveit_config)/config/robotiq_gripper.srdf.xacro" />
     <xacro:robotiq_gripper side="left"/>
+    REVERT 1-->
   </xacro:if>
   <!--Right End Effector Collisions-->

File: setup/Backup/baxter_moveit_config/config/gazebo_baxter.urdf (robot description, URDF)
Before this commit: robot baxter, 62 links, 61 joints
Links:
- removed link robotiq_arg2f_base_link
- added link left_gripper, mass 0.22652; collision mesh filename=package://robotiq_2f_85_gripper_vis/meshes/collision/roboti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; visual mesh filename=package://robotiq_2f_85_gripper_vis/meshes/visual/robotiq_a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 scale=0.001 0.001 0.001
- link display: geometry collision box size=0.218 0.16 0.001; visual box size=0.218 0.16 0.001
- link left_hand_accelerometer: geometry collision box size=0.01 0.01 0.01; visual box size=0.01 0.01 0.01
- link left_hand_camera: geometry collision cylinder length=0.01 radius=0.02; visual cylinder length=0.01 radius=0.02
- link left_hand_range: geometry collision box size=0.005 0.02 0.005; visual box size=0.005 .02 .005
- link right_hand_accelerometer: geometry collision box size=0.01 0.01 0.01; visual box size=0.01 0.01 0.01
- link right_hand_camera: geometry collision cylinder length=0.01 radius=0.02; visual cylinder length=0.01 radius=0.02
- link right_hand_range: geometry collision box size=0.005 .02 .005; visual box size=0.005 .02 .005
Joints:
- joint finger_joint: parent robotiq_arg2f_base_link -> left_gripper
- joint left_inner_knuckle_joint: parent robotiq_arg2f_base_link -> left_gripper
- joint right_inner_knuckle_joint: parent robotiq_arg2f_base_link -> left_gripper
- joint right_outer_knuckle_joint: parent robotiq_arg2f_base_link -> left_gripper
- joint robotiq_arg2f_base_joint: child robotiq_arg2f_base_link -> left_gripper

File: setup/Backup/baxter_moveit_config/config/rethink_electric_gripper.srdf.xacro (robot description, xacro)
@@ -16,7 +16,14 @@
     <disable_collisions link1="${side}_gripper" link2="${gripper_side}_gripper_r_finger" reason="Default" />
     <disable_collisions link1="${side}_gripper" link2="${gripper_side}_gripper_r_finger_tip" reason="Never" />
-    <disable_collisions link1="${gripper_side}_gripper_l_finger" link2="${gripper_side}_gripper_l_finger_tip" reason="Adjacent" />
+    <!-- Between links -->
+    <disable_collisions link1="${gripper_side}_gripper_l_finger" link2="${gripper_side}_gripper_r_finger_tip" reason="Adjacent" />
     <disable_collisions link1="${gripper_side}_gripper_l_finger" link2="${gripper_side}_gripper_r_finger" reason="Never" />
     <disable_collisions link1="${gripper_side}_gripper_l_finger" link2="${gripper_side}_gripper_r_finger_tip" reason="Never" />
+    <disable_collisions link1="${gripper_side}_gripper_l_finger_tip" link2="${gripper_side}_gripper_r_finger" reason="Never" />
+    <disable_collisions link1="${gripper_side}_gripper_r_finger" link2="${gripper_side}_gripper_r_finger_tip" reason="Adjacent" />
+    <disable_collisions link1="${gripper_side}_gripper_l_finger_tip" link2="${gripper_side}_gripper_r_finger_tip" reason="Never" />
+    <disable_collisions link1="${gripper_side}_gripper_l_finger" link2="${gripper_side}_gripper_l_finger_tip" reason="Never" />
+    <disable_collisions link1="${gripper_side}_gripper_r_finger" link2="${gripper_side}_gripper_r_finger_tip" reason="Never" />
+    <!-- l -->
     <disable_collisions link1="${gripper_side}_gripper_l_finger" link2="${side}_hand" reason="Never" />
     <disable_collisions link1="${gripper_side}_gripper_l_finger" link2="${side}_hand_accelerometer" reason="Never" />
@@ -28,5 +35,4 @@
     <disable_collisions link1="${gripper_side}_gripper_l_finger" link2="${side}_upper_forearm_visual" reason="Never" />
     <disable_collisions link1="${gripper_side}_gripper_l_finger" link2="${side}_wrist" reason="Never" />
-    <disable_collisions link1="${gripper_side}_gripper_l_finger_tip" link2="${gripper_side}_gripper_r_finger" reason="Never" />
     <disable_collisions link1="${gripper_side}_gripper_l_finger_tip" link2="${side}_hand" reason="Never" />
     <disable_collisions link1="${gripper_side}_gripper_l_finger_tip" link2="${side}_hand_accelerometer" reason="Never" />
@@ -39,5 +45,5 @@
     <disable_collisions link1="${gripper_side}_gripper_l_finger_tip" link2="${side}_upper_forearm_visual" reason="Never" />
     <disable_collisions link1="${gripper_side}_gripper_l_finger_tip" link2="${side}_wrist" reason="Never" />
-    <disable_collisions link1="${gripper_side}_gripper_r_finger" link2="${gripper_side}_gripper_r_finger_tip" reason="Adjacent" />
+    <!-- r -->
     <disable_collisions link1="${gripper_side}_gripper_r_finger" link2="${side}_hand" reason="Never" />
     <disable_collisions link1="${gripper_side}_gripper_r_finger" link2="${side}_hand_accelerometer" reason="Never" />
@@ -59,7 +65,4 @@
     <disable_collisions link1="${gripper_side}_gripper_r_finger_tip" link2="${side}_upper_forearm_visual" reason="Never" />
     <disable_collisions link1="${gripper_side}_gripper_r_finger_tip" link2="${side}_wrist" reason="Never" />
-    <disable_collisions link1="${gripper_side}_gripper_l_finger_tip" link2="${gripper_side}_gripper_r_finger_tip" reason="Never" />
-    <disable_collisions link1="${gripper_side}_gripper_l_finger" link2="${gripper_side}_gripper_l_finger_tip" reason="Never" />
-    <disable_collisions link1="${gripper_side}_gripper_r_finger" link2="${gripper_side}_gripper_r_finger_tip" reason="Never" />
     </xacro:macro>
 </robot>

File: setup/Backup/baxter_moveit_config/config/robotiq_gripper.srdf.xacro (robot description, xacro)
@@ -5,66 +5,25 @@
 -->
 <robot xmlns:xacro="http://www.ros.org/wiki/xacro" name="robotiq_gripper">
-    <!-- Macro for robotiq_gripper Gripper (Left) FOR NOW -->
-    <xacro:macro name="robotiq_arg2f_85_model_macro">
-    <xacro:property name="gripper_side" value="l" scope="local"/> <!-- "l" is for left side -->
-    <!-- robotiq_arg2f_base_link -->
-    <disable_collisions link1="robotiq_arg2f_base_link" link2="${gripper_side}_gripper_l_finger" reason="Adjacent" />
-    <disable_collisions link1="robotiq_arg2f_base_link" link2="${gripper_side}_gripper_l_finger_tip" reason="Never" />
-    <disable_collisions link1="${side}_gripper_base" link2="${gripper_side}_gripper_r_finger" reason="Adjacent" />
-    <disable_collisions link1="${side}_gripper_base" link2="${gripper_side}_gripper_r_finger_tip" reason="Never" />
-    <!--  -->
-    <disable_collisions link1="${side}_gripper" link2="${gripper_side}_gripper_l_finger" reason="Default" />
-    <disable_collisions link1="${side}_gripper" link2="${gripper_side}_gripper_l_finger_tip" reason="Never" />
-    <disable_collisions link1="${side}_gripper" link2="${gripper_side}_gripper_r_finger" reason="Default" />
-    <disable_collisions link1="${side}_gripper" link2="${gripper_side}_gripper_r_finger_tip" reason="Never" />
-    <!--  -->
-    <disable_collisions link1="${gripper_side}_gripper_l_finger" link2="${gripper_side}_gripper_l_finger_tip" reason="Adjacent" />
-    <disable_collisions link1="${gripper_side}_gripper_l_finger" link2="${gripper_side}_gripper_r_finger" reason="Never" />
-    <disable_collisions link1="${gripper_side}_gripper_l_finger" link2="${gripper_side}_gripper_r_finger_tip" reason="Never" />
-    <disable_collisions link1="${gripper_side}_gripper_l_finger" link2="${side}_hand" reason="Never" />
-    <disable_collisions link1="${gripper_side}_gripper_l_finger" link2="${side}_hand_accelerometer" reason="Never" />
-    <disable_collisions link1="${gripper_side}_gripper_l_finger" link2="${side}_hand_camera" reason="Never" />
-    <disable_collisions link1="${gripper_side}_gripper_l_finger" link2="${side}_hand_range" reason="Never" />
-    <disable_collisions link1="${gripper_side}_gripper_l_finger" link2="${side}_lower_elbow" reason="Never" />
-    <disable_collisions link1="${gripper_side}_gripper_l_finger" link2="${side}_lower_forearm" reason="Never" />
-    <disable_collisions link1="${gripper_side}_gripper_l_finger" link2="${side}_upper_forearm" reason="Never" />
-    <disable_collisions link1="${gripper_side}_gripper_l_finger" link2="${side}_upper_forearm_visual" reason="Never" />
-    <disable_collisions link1="${gripper_side}_gripper_l_finger" link2="${side}_wrist" reason="Never" />
-    <disable_collisions link1="${gripper_side}_gripper_l_finger_tip" link2="${gripper_side}_gripper_r_finger" reason="Never" />
-    <disable_collisions link1="${gripper_side}_gripper_l_finger_tip" link2="${side}_hand" reason="Never" />
-    <disable_collisions link1="${gripper_side}_gripper_l_finger_tip" link2="${side}_hand_accelerometer" reason="Never" />
-    <disable_collisions link1="${gripper_side}_gripper_l_finger_tip" link2="${side}_hand_camera" reason="Never" />
-    <disable_collisions link1="${gripper_side}_gripper_l_finger_tip" link2="${side}_hand_range" reason="Never" />
-    <disable_collisions link1="${gripper_side}_gripper_l_finger_tip" link2="${side}_lower_elbow" reason="Never" />
-    <disable_collisions link1="${gripper_side}_gripper_l_finger_tip" link2="${side}_lower_forearm" reason="Never" />
-    <disable_collisions link1="${gripper_side}_gripper_l_finger_tip" link2="${side}_upper_elbow_visual" reason="Never" />
-    <disable_collisions link1="${gripper_side}_gripper_l_finger_tip" link2="${side}_upper_forearm" reason="Never" />
-    <disable_collisions link1="${gripper_side}_gripper_l_finger_tip" link2="${side}_upper_forearm_visual" reason="Never" />
-    <disable_collisions link1="${gripper_side}_gripper_l_finger_tip" link2="${side}_wrist" reason="Never" />
-    <!--  -->
-    <disable_collisions link1="${gripper_side}_gripper_r_finger" link2="${gripper_side}_gripper_r_finger_tip" reason="Adjacent" />
-    <disable_collisions link1="${gripper_side}_gripper_r_finger" link2="${side}_hand" reason="Never" />
-    <disable_collisions link1="${gripper_side}_gripper_r_finger" link2="${side}_hand_accelerometer" reason="Never" />
-    <disable_collisions link1="${gripper_side}_gripper_r_finger" link2="${side}_hand_camera" reason="Never" />
-    <disable_collisions link1="${gripper_side}_gripper_r_finger" link2="${side}_hand_range" reason="Never" />
-    <disable_collisions link1="${gripper_side}_gripper_r_finger" link2="${side}_lower_elbow" reason="Never" />
-    <disable_collisions link1="${gripper_side}_gripper_r_finger" link2="${side}_lower_forearm" reason="Never" />
-    <disable_collisions link1="${gripper_side}_gripper_r_finger" link2="${side}_upper_forearm" reason="Never" />
-    <disable_collisions link1="${gripper_side}_gripper_r_finger" link2="${side}_upper_forearm_visual" reason="Never" />
-    <disable_collisions link1="${gripper_side}_gripper_r_finger" link2="${side}_wrist" reason="Never" />
-    <disable_collisions link1="${gripper_side}_gripper_r_finger_tip" link2="${side}_hand" reason="Never" />
-    <disable_collisions link1="${gripper_side}_gripper_r_finger_tip" link2="${side}_hand_accelerometer" reason="Never" />
-    <disable_collisions link1="${gripper_side}_gripper_r_finger_tip" link2="${side}_hand_camera" reason="Never" />
-    <disable_collisions link1="${gripper_side}_gripper_r_finger_tip" link2="${side}_hand_range" reason="Never" />
-    <disable_collisions link1="${gripper_side}_gripper_r_finger_tip" link2="${side}_lower_elbow" reason="Never" />
-    <disable_collisions link1="${gripper_side}_gripper_r_finger_tip" link2="${side}_lower_forearm" reason="Never" />
-    <disable_collisions link1="${gripper_side}_gripper_r_finger_tip" link2="${side}_upper_elbow_visual" reason="Never" />
-    <disable_collisions link1="${gripper_side}_gripper_r_finger_tip" link2="${side}_upper_forearm" reason="Never" />
-    <disable_collisions link1="${gripper_side}_gripper_r_finger_tip" link2="${side}_upper_forearm_visual" reason="Never" />
-    <disable_collisions link1="${gripper_side}_gripper_r_finger_tip" link2="${side}_wrist" reason="Never" />
-    <!--  -->
-    <disable_collisions link1="${gripper_side}_gripper_l_finger_tip" link2="${gripper_side}_gripper_r_finger_tip" reason="Never" />
-    <disable_collisions link1="${gripper_side}_gripper_l_finger" link2="${gripper_side}_gripper_l_finger_tip" reason="Never" />
-    <disable_collisions link1="${gripper_side}_gripper_r_finger" link2="${gripper_side}_gripper_r_finger_tip" reason="Never" />
+    <xacro:macro name="robotiq_gripper" params="side"> <!-- fingerprefix is like side[0]-->
+    <!-- Disable collision between two specific links: link1 and link2 -->
+    <disable_collisions link1="left_gripper" link2="left_inner_finger_pad" reason="Never" />
+    <disable_collisions link1="left_gripper" link2="left_inner_finger" reason="Never" />
+    <disable_collisions link1="left_gripper" link2="left_inner_knuckle" reason="Never" />
+    <disable_collisions link1="left_gripper" link2="left_outer_finger" reason="Never" />
+    <disable_collisions link1="left_gripper" link2="left_outer_knuckle" reason="Never" />
+    <disable_collisions link1="left_gripper" link2="right_inner_finger_pad" reason="Never" />
+    <disable_collisions link1="left_gripper" link2="right_inner_finger" reason="Never" />
+    <disable_collisions link1="left_gripper" link2="right_inner_knuckle" reason="Never" />
+    <disable_collisions link1="left_gripper" link2="right_outer_finger" reason="Never" />
+    <disable_collisions link1="left_gripper" link2="right_outer_knuckle" reason="Never" />
+    <disable_collisions link1="left_gripper" link2="${side}_hand" reason="Never" />
+    <disable_collisions link1="left_gripper" link2="${side}_hand_accelerometer" reason="Never" />
+    <disable_collisions link1="left_gripper" link2="${side}_hand_camera" reason="Never" />
+    <disable_collisions link1="left_gripper" link2="${side}_hand_range" reason="Never" />
+    <disable_collisions link1="left_gripper" link2="${side}_lower_elbow" reason="Never" />
+    <disable_collisions link1="left_gripper" link2="${side}_lower_forearm" reason="Never" />
+    <disable_collisions link1="left_gripper" link2="${side}_upper_forearm" reason="Never" />
+    <disable_collisions link1="left_gripper" link2="${side}_upper_forearm_visual" reason="Never" />
+    <disable_collisions link1="left_gripper" link2="${side}_wrist" reason="Never" />
     </xacro:macro>
 </robot>

File: ws_AF/src/baxter_common/baxter_description/urdf/baxter.urdf (robot description, URDF)
Before this commit: robot baxter, 62 links, 61 joints
Links:
- link display: geometry collision box size=0.218 0.16 0.001; visual box size=0.218 0.16 0.001
- link left_hand_accelerometer: geometry collision box size=0.01 0.01 0.01; visual box size=0.01 0.01 0.01
- link left_hand_camera: geometry collision cylinder length=0.01 radius=0.02; visual cylinder length=0.01 radius=0.02
- link left_hand_range: geometry collision box size=0.005 0.02 0.005; visual box size=0.005 .02 .005
- link right_hand_accelerometer: geometry collision box size=0.01 0.01 0.01; visual box size=0.01 0.01 0.01
- link right_hand_camera: geometry collision cylinder length=0.01 radius=0.02; visual cylinder length=0.01 radius=0.02
- link right_hand_range: geometry collision box size=0.005 .02 .005; visual box size=0.005 .02 .005

File: ws_AF/src/baxter_common/baxter_description/urdf/baxter_base/baxter_base.urdf.xacro (robot description, xacro)
@@ -120,4 +120,10 @@
       </material>
     </visual>
+    <collision>
+      <origin rpy="0.2617993877991494 0 0" xyz="0 0 0"/>
+      <geometry>
+        <box size="0.218 0.16 0.001"/>
+      </geometry>
+    </collision>
     <inertial>
       <origin rpy="0 0 0" xyz="0 0 0"/>
@@ -462,4 +468,10 @@
       </material>
     </visual>
+    <collision>
+      <origin rpy="0 0 0" xyz="0 0 0"/>
+      <geometry>
+        <cylinder length="0.01" radius="0.02"/>
+      </geometry>
+    </collision>
     <inertial>
       <origin rpy="0 0 0" xyz="0 0 0"/>
@@ -485,4 +497,10 @@
       </material>
     </visual>
+    <collision>
+      <origin rpy="0 0 0" xyz="0 0 0"/>
+      <geometry>
+        <box size="0.005 .02 .005"/>
+      </geometry>
+    </collision>
     <inertial>
       <origin rpy="0 0 0" xyz="0 0 0"/>
@@ -501,4 +519,10 @@
       </material>
     </visual>
+    <collision>
+      <origin rpy="0 0 0" xyz="0 0 0"/>
+      <geometry>
+        <box size="0.01 0.01 0.01"/>
+      </geometry>
+    </collision>
     <inertial>
       <origin rpy="0 0 0" xyz="0.000000 0.000000 0.000000"/>
@@ -830,4 +854,10 @@
       </material>
     </visual>
+    <collision>
+      <origin rpy="0 0 0" xyz="0 0 0"/>
+      <geometry>
+        <cylinder length="0.01" radius="0.02"/>
+      </geometry>
+    </collision>
     <inertial>
       <origin rpy="0 0 0" xyz="0 0 0"/>
@@ -853,4 +883,10 @@
       </material>
     </visual>
+    <collision>
+      <origin rpy="0 0 0" xyz="0 0 0"/>
+      <geometry>
+        <box size="0.005 0.02 0.005"/>
+      </geometry>
+    </collision>
     <inertial>
       <origin rpy="0 0 0" xyz="0 0 0"/>
@@ -869,4 +905,10 @@
       </material>
     </visual>
+    <collision>
+      <origin rpy="0 0 0" xyz="0 0 0"/>
+      <geometry>
+        <box size="0.01 0.01 0.01"/>
+      </geometry>
+    </collision>
     <inertial>
       <origin rpy="0 0 0" xyz="0.000000 0.000000 0.000000"/>

File: ws_AF/src/moveit_robots/baxter_moveit_config/baxter_moveit_config/config/baxter.srdf.xacro (robot description, xacro)
@@ -1,9 +1,6 @@
 <?xml version="1.0" ?>
 <robot name="baxter" xmlns:xacro="http://www.ros.org/wiki/xacro">
-  <!-- Arguments (go into baxter_base)-->
   <xacro:arg name="left_tip_name" default="left_gripper"/>
   <xacro:arg name="right_tip_name" default="right_gripper"/>
-  <!--<xacro:arg name="left_robotiq_gripper" default="false"/> -->
-  <!-- Base Configuration -->
   <xacro:include filename="$(find baxter_moveit_config)/config/baxter_base.srdf.xacro" />
   <xacro:baxter_base left_tip_name="$(arg left_tip_name)" right_tip_name="$(arg right_tip_name)"/>
@@ -12,9 +9,4 @@
   <xacro:left_default_gripper side="left"/>
   <xacro:arg name="left_electric_gripper" default="false"/>
-  <!-- <xacro:if value="$(arg left_electric_gripper)">
-    <xacro:include filename="$(find baxter_moveit_config)/config/rethink_electric_gripper.srdf.xacro" />
-    <xacro:rethink_electric_gripper side="left"/>
-  </xacro:if> -->
-  <!-- Conditional inclusion of Robotiq gripper -->
   <xacro:if value="$(arg left_electric_gripper)">
     <xacro:include filename="$(find baxter_moveit_config)/config/robotiq_gripper.srdf.xacro" />

File: ws_AF/src/moveit_robots/baxter_moveit_config/baxter_moveit_config/config/baxter_base.srdf.xacro (robot description, xacro)
@@ -5,5 +5,5 @@
 -->
 <robot xmlns:xacro="http://www.ros.org/wiki/xacro" name="baxter">
-  <xacro:macro name="baxter_base" params="left_tip_name right_tip_name"> <!-- left_gripper, right_gripper -->
+  <xacro:macro name="baxter_base" params="left_tip_name right_tip_name">
     <!--GROUPS: Representation of a set of joints and links. This can be useful for specifying DOF to plan for, defining arms, end effectors, etc-->
     <!--LINKS: When a link is specified, the parent joint of that link (if it exists) is automatically included-->
