Commit message: Currently working in Moveit

File: ws_AF/src/baxter_common/baxter_description/urdf/baxter.urdf (robot description, URDF)
Before this commit: robot baxter, 62 links, 61 joints
Links:
- added link left_gripper_base, mass 0.22652; collision mesh filename=package://robotiq_2f_85_gripper_vis/meshes/collision/roboti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; visual mesh filename=package://robotiq_2f_85_gripper_vis/meshes/visual/robotiq_a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 scale=0.001 0.001 0.001
- link left_gripper: mass 0.22652 -> 0.0001; geometry 
Joints:
- removed joint finger_joint
- removed joint robotiq_arg2f_base_joint
- added joint left_endpoint: type fixed, parent left_gripper_base, child left_gripper, origin xyz=0 0 0.15032399999999999 rpy=0 0 0
- added joint left_gripper_base: type fixed, parent left_hand, child left_gripper_base, origin xyz=0 0 0 rpy=0 0 0, axis 0 0 1
- added joint left_outer_knuckle_joint: type revolute, parent left_gripper_base, child left_outer_knuckle, origin xyz=0 -0.0306011 0.054904 rpy=0 0 3.141592653589793, axis 1 0 0, limit lower=0 upper=0.8 effort=1000 velocity=2.0
- joint left_inner_finger_joint: mimic joint=finger_joint multiplier=-1 offset=0 -> joint=left_outer_knuckle_joint multiplier=-1 offset=0
- joint left_inner_knuckle_joint: mimic joint=finger_joint multiplier=1 offset=0 -> joint=left_outer_knuckle_joint multiplier=1 offset=0; parent left_gripper -> left_gripper_base
- joint right_inner_finger_joint: mimic joint=finger_joint multiplier=-1 offset=0 -> joint=left_outer_knuckle_joint multiplier=-1 offset=0
- joint right_inner_knuckle_joint: mimic joint=finger_joint multiplier=1 offset=0 -> joint=left_outer_knuckle_joint multiplier=1 offset=0; parent left_gripper -> left_gripper_base
- joint right_outer_knuckle_joint: mimic joint=finger_joint multiplier=1 offset=0 -> joint=left_outer_knuckle_joint multiplier=1 offset=0; parent left_gripper -> left_gripper_base

File: ws_AF/src/baxter_common/baxter_description/urdf/left_end_effector.urdf.xacro (robot description, xacro)
@@ -3,4 +3,4 @@
   <!-- Include the Robotiq 2F-85 gripper Xacro file -->
   <xacro:include filename="$(find robotiq_2f_85_gripper_vis)/urdf/robotiq_arg2f_85_model_macro.xacro" />
-  <xacro:left_gripper prefix="" /> <!-- loads the model in -->
+  <xacro:left_gripper_base prefix="" /> <!-- loads the model in -->
 </robot>

File: ws_AF/src/baxter_common/robotiq_2f_85_gripper_vis/urdf/robotiq_arg2f.xacro (robot description, xacro)
@@ -3,5 +3,5 @@
   <!-- Robotiq Gripper Base Link -->
   <xacro:macro name="robotiq_arg2f_base_link" params="prefix">
-    <link name="left_gripper"> <!-- OLD: ${prefix}robotiq_arg2f_base_link -->
+    <link name="left_gripper_base"> <!-- OLD: ${prefix}robotiq_arg2f_base_link -->
       <inertial>
         <origin xyz="8.625E-08 -4.6583E-06 0.03145" rpy="0 0 0" />
@@ -25,11 +25,25 @@
       </collision>
     </link>
-    <joint name="${prefix}robotiq_arg2f_base_joint" type="fixed">
-      <origin xyz="0 0 0" rpy="0 0 0.11355"/>  <!-- Adjust if there is an offset between the gripper and Baxter's end effector -->
+    <joint name="left_gripper_base" type="fixed">
+      <origin xyz="0 0 0" rpy="0 0 0"/>  <!-- Adjust if there is an offset between the gripper and Baxter's end effector -->
       <axis xyz="0 0 1"/>
       <parent link="left_hand"/>  <!-- Replace with the actual Baxter end effector link name -->
-      <child link="left_gripper"/> <!-- changed with new name -->
+      <child link="left_gripper_base"/> <!-- changed with new name -->
   </joint>
   </xacro:macro>
+  <!-- Electric Gripper Tip joint -->
+  <joint name="left_endpoint" type="fixed">
+    <origin rpy="0 0 0" xyz="0 0 ${0.130324+0.02}"/> <!-- Value added from all z values manually-->
+    <parent link="left_gripper_base"/>
+    <child link="left_gripper"/>
+  </joint>
+  <!-- Electric Gripper Tip link -->
+  <link name="left_gripper">
+    <inertial>
+      <origin rpy="0 0 0" xyz="0 0 0"/>
+      <mass value="0.0001"/>
+      <inertia ixx="0" ixy="0" ixz="0" iyy="0" iyz="0" izz="0.0"/>
+    </inertial>
+  </link>
   <xacro:macro name="finger_joints" params="prefix fingerprefix reflect">
     <xacro:outer_finger_joint prefix="${prefix}" fingerprefix="${fingerprefix}"/>

File: ws_AF/src/baxter_common/robotiq_2f_85_gripper_vis/urdf/robotiq_arg2f_85_model_macro.xacro (robot description, xacro)
@@ -133,9 +133,9 @@
       <!-- <origin xyz="0 ${reflect * -0.0127} 0.06142" rpy="${pi / 2 + .725} 0 ${(reflect - 1) * pi / 2}" /> -->
       <origin xyz="0 ${reflect * -0.0127} 0.06142" rpy="0 0 ${(1 + reflect) * pi / 2}"/>
-      <parent link="left_gripper" /> <!-- changed with name change-->
+      <parent link="left_gripper_base" /> <!-- changed with name change-->
       <child link="${prefix}${fingerprefix}_inner_knuckle" />
       <axis xyz="1 0 0" />
       <limit lower="0" upper="0.8757" velocity="2.0" effort="1000" />
-      <mimic joint="${prefix}finger_joint" multiplier="1" offset="0" />
+      <mimic joint="${prefix}left_outer_knuckle_joint" multiplier="1" offset="0" />
     </joint>
   </xacro:macro>
@@ -147,5 +147,5 @@
       <axis xyz="1 0 0" />
       <limit lower="0" upper="0.8757" velocity="2.0" effort="1000" />
-      <mimic joint="${prefix}finger_joint" multiplier="-1" offset="0" />
+      <mimic joint="${prefix}left_outer_knuckle_joint" multiplier="-1" offset="0" />
     </joint>
   </xacro:macro>
@@ -160,8 +160,8 @@
   <!-- LOADS FROM THE OTHER FILE -->
   <xacro:include filename="$(find robotiq_2f_85_gripper_vis)/urdf/robotiq_arg2f.xacro" />
-  <xacro:macro name="finger_joint" params="prefix">
-    <joint name="${prefix}finger_joint" type="revolute">
+  <xacro:macro name="left_outer_knuckle_joint" params="prefix">
+    <joint name="${prefix}left_outer_knuckle_joint" type="revolute">
       <origin xyz="0 -0.0306011 0.054904" rpy="0 0 ${pi}"/>
-      <parent link="left_gripper" /> <!-- changed with name change for base-->
+      <parent link="left_gripper_base" /> <!-- changed with name change for base-->
       <child link="${prefix}left_outer_knuckle" />
       <axis xyz="1 0 0" />
@@ -173,19 +173,19 @@
     <joint name="${prefix}right_outer_knuckle_joint" type="revolute">
       <origin xyz="0 0.0306011 0.054904" rpy="0 0 0"/>
-      <parent link="left_gripper" /> <!-- changed with base name change -->
+      <parent link="left_gripper_base" /> <!-- changed with base name change -->
       <child link="${prefix}right_outer_knuckle" />
       <axis xyz="1 0 0" />
       <limit lower="0" upper="0.81" velocity="2.0" effort="1000" />
-      <mimic joint="${prefix}finger_joint" multiplier="1" offset="0" />
+      <mimic joint="${prefix}left_outer_knuckle_joint" multiplier="1" offset="0" />
     </joint>
     <xacro:finger_joints prefix="${prefix}" fingerprefix="right" reflect="-1.0"/>
   </xacro:macro>
   <!-- Initialization of all joints and links -->
-  <xacro:macro name="left_gripper" params="prefix">
+  <xacro:macro name="left_gripper_base" params="prefix">
     <xacro:robotiq_arg2f_base_link prefix="${prefix}"/>
     <xacro:finger_links prefix="${prefix}" fingerprefix="left" stroke="85"/>
     <xacro:finger_links prefix="${prefix}" fingerprefix="right" stroke="85"/>
-    <xacro:finger_joint prefix="${prefix}"/>
     <xacro:right_outer_knuckle_joint prefix="${prefix}"/>
+    <xacro:left_outer_knuckle_joint prefix="${prefix}"/>
     <xacro:robotiq_arg2f_transmission prefix="${prefix}"/>
   </xacro:macro>
