Commit message: Chnages made to implement the Barrett Hand. Barrett hand not working Robotiq is

File: ws_AF/src/baxter_common/baxter_description/urdf/baxter.urdf (robot description, URDF)
Before this commit: robot baxter, 63 links, 62 joints
Links:
- removed link r_gripper_l_finger
- removed link r_gripper_l_finger_tip
- removed link r_gripper_r_finger
- removed link r_gripper_r_finger_tip
- removed link right_gripper
- removed link right_gripper_base
- added link barrett_base_link, mass 0.1; collision mesh filename=package://barrett_hand_vis/meshes/base_link.STL; visual mesh filename=package://barrett_hand_vis/meshes/base_link.STL
- added link finger_1_dist_link, mass 0.001; collision mesh filename=package://barrett_hand_vis/meshes/finger_1_dist_link.STL; visual mesh filename=package://barrett_hand_vis/meshes/finger_1_dist_link.STL
- added link finger_1_med_link, mass 0.1; collision mesh filename=package://barrett_hand_vis/meshes/finger_1_med_link.STL; visual mesh filename=package://barrett_hand_vis/meshes/finger_1_med_link.STL
- added link finger_1_prox_link, mass 0.1; collision mesh filename=package://barrett_hand_vis/meshes/finger_1_prox_link.STL; visual mesh filename=package://barrett_hand_vis/meshes/finger_1_prox_link.STL
- added link finger_2_dist_link, mass 0.001; collision mesh filename=package://barrett_hand_vis/meshes/finger_2_dist_link.STL; visual mesh filename=package://barrett_hand_vis/meshes/finger_2_dist_link.STL
- added link finger_2_med_link, mass 0.1; collision mesh filename=package://barrett_hand_vis/meshes/finger_2_med_link.STL; visual mesh filename=package://barrett_hand_vis/meshes/finger_2_med_link.STL
- added link finger_2_prox_link, mass 0.1; collision mesh filename=package://barrett_hand_vis/meshes/finger_2_prox_link.STL; visual mesh filename=package://barrett_hand_vis/meshes/finger_2_prox_link.STL
- added link finger_3_dist_link, mass 0.1; collision mesh filename=package://barrett_hand_vis/meshes/finger_3_dist_link.STL; visual mesh filename=package://barrett_hand_vis/meshes/finger_3_dist_link.STL
- added link finger_3_med_link, mass 0.1; collision mesh filename=package://barrett_hand_vis/meshes/finger_3_med_link.STL; visual mesh filename=package://barrett_hand_vis/meshes/finger_3_med_link.STL
- added link palm_frame
Joints:
- removed joint left_endpoint
- removed joint left_outer_knuckle_joint
- removed joint r_gripper_l_finger_joint
- removed joint r_gripper_l_finger_tip_joint
- removed joint r_gripper_r_finger_joint
- removed joint r_gripper_r_finger_tip_joint
- removed joint right_endpoint
- removed joint right_gripper_base
- added joint base_joint: type fixed, parent right_hand, child barrett_base_link, origin xyz=0 0 0.002 rpy=0 0 4.7124
- added joint finger_1_dist_joint: type revolute, parent finger_1_med_link, child finger_1_dist_link, origin xyz=-0.069936 -0.003 0 rpy=1.6787E-18 -3.6382E-15 -6.1073E-33, axis 0 0 1, limit lower=0.6 upper=1.57 effort=10000 velocity=0.2, mimic joint=finger_1_med_joint multiplier=0.3 offset=0.75
- added joint finger_1_med_joint: type revolute, parent finger_1_prox_link, child finger_1_med_link, origin xyz=-0.05 0 0.0339 rpy=-1.5708 -8.8281E-17 0, axis 0 0 1, limit lower=0 upper=2.44 effort=10000 velocity=0.2
- added joint finger_1_prox_joint: type revolute, parent barrett_base_link, child finger_1_prox_link, origin xyz=0.025 0 0.0415 rpy=0 2.7051E-17 -1.5708, axis 0 0 -1, limit lower=0.0 upper=3.141 effort=10000 velocity=0.2
- added joint finger_2_dist_joint: type revolute, parent finger_2_med_link, child finger_2_dist_link, origin xyz=-0.069917 -0.0034087 0 rpy=-3.1382E-17 -2.3229E-16 0, axis 0 0 1, limit lower=0.6 upper=1.57 effort=10000 velocity=0.2, mimic joint=finger_2_med_joint multiplier=0.3 offset=0.75
- added joint finger_2_med_joint: type revolute, parent finger_2_prox_link, child finger_2_med_link, origin xyz=-0.05 0 0.0339 rpy=-1.5708 -8.8281E-17 0, axis 0 0 1, limit lower=0.0 upper=2.44 effort=10000 velocity=0.2
- added joint finger_2_prox_joint: type revolute, parent barrett_base_link, child finger_2_prox_link, origin xyz=-0.025 0 0.0415 rpy=0 2.7051E-17 -1.5708, axis 0 0 1, limit lower=0 upper=3.141 effort=10000 velocity=0.2
- added joint finger_3_dist_joint: type revolute, parent finger_3_med_link, child finger_3_dist_link, origin xyz=-0.069936 -0.003 0 rpy=6.0427E-17 -6.7283E-18 -4.0657E-34, axis 0 0 1, limit lower=0.6 upper=1.57 effort=10000 velocity=0.2, mimic joint=finger_3_med_joint multiplier=0.3 offset=0.75
- added joint finger_3_med_joint: type revolute, parent barrett_base_link, child finger_3_med_link, origin xyz=0 -0.05 0.0754 rpy=-1.5708 6.123E-17 1.5708, axis 0 0 1, limit lower=0.0 upper=2.44 effort=10000 velocity=0.2
- added joint finger_joint: type revolute, parent left_gripper_base, child left_outer_knuckle, origin xyz=0 -0.0306011 0.054904 rpy=0 0 3.141592653589793, axis 1 0 0, limit lower=0 upper=0.8 effort=1000 velocity=2.0
- added joint left_endpoint_joint: type fixed, parent left_gripper_base, child left_gripper, origin xyz=0 0 0.15032399999999999 rpy=0 0 0
- added joint palm_joint: type fixed, parent barrett_base_link, child palm_frame, origin xyz=0.0 0.0 0.077
- joint left_inner_finger_joint: mimic joint=left_outer_knuckle_joint multiplier=-1 offset=0 -> joint=finger_joint multiplier=-1 offset=0
- joint left_inner_knuckle_joint: mimic joint=left_outer_knuckle_joint multiplier=1 offset=0 -> joint=finger_joint multiplier=1 offset=0
- joint right_inner_finger_joint: mimic joint=left_outer_knuckle_joint multiplier=-1 offset=0 -> joint=finger_joint multiplier=-1 offset=0
- joint right_inner_knuckle_joint: mimic joint=left_outer_knuckle_joint multiplier=1 offset=0 -> joint=finger_joint multiplier=1 offset=0
- joint right_outer_knuckle_joint: mimic joint=left_outer_knuckle_joint multiplier=1 offset=0 -> joint=finger_joint multiplier=1 offset=0

File: ws_AF/src/baxter_common/baxter_description/urdf/left_end_effector.urdf.xacro (robot description, xacro)
@@ -1,6 +1,9 @@
 <?xml version="1.0" ?>
 <robot name="left_end_effector" xmlns:xacro="http://www.ros.org/wiki/xacro">
+  <!-- Define necessary properties for the gripper -->
+  <xacro:property name="dist_joint_multiplier" value="0.3" />
+  <xacro:property name="dist_joint_offset" value="0.75" />
   <!-- Include the Robotiq 2F-85 gripper Xacro file -->
   <xacro:include filename="$(find robotiq_2f_85_gripper_vis)/urdf/robotiq_arg2f_85_model_macro.xacro" />
-  <xacro:left_gripper_base prefix="" /> <!-- loads the model in -->
+  <xacro:left_robotiq_gripper prefix="" /> <!-- loads the model in -->
 </robot>

File: ws_AF/src/baxter_common/baxter_description/urdf/right_end_effector.urdf.xacro (robot description, xacro)
@@ -1,13 +1,15 @@
 <?xml version="1.0" ?>
 <robot name="right_end_effector" xmlns:xacro="http://www.ros.org/wiki/xacro">
-  <xacro:include filename="$(find rethink_ee_description)/urdf/electric_gripper/rethink_electric_gripper.xacro" />
-  <xacro:rethink_electric_gripper side="right"
-                                  l_finger="extended_narrow"
-                                  l_finger_slot="2"
-                                  l_finger_tip="half_round_tip"
-                                  l_finger_grasp="inner"
-                                  r_finger="extended_narrow"
-                                  r_finger_slot="2"
-                                  r_finger_tip="half_round_tip"
-                                  r_finger_grasp="inner"/>
+  <!-- <xacro:include filename="$(find barrett_hand_vis)/urdf/bh282.urdf.xacro" />
+  <xacro:bhand_macro name="bh" parent="right_hand">
+    <origin xyz="0 0 0.5" rpy="0 0 0" />
+  </xacro:bhand_macro> -->
+  <!-- Import Rviz colors -->
+  <xacro:include filename="$(find barrett_hand_vis)/urdf/materials.xacro" />
+  <joint name="base_joint" type="fixed">
+    <origin xyz="0 0 0.002" rpy="0 0 4.7124"/>
+    <parent link="right_hand"/>
+    <child link="barrett_base_link"/>
+  </joint>
+  <xacro:include filename="$(find barrett_hand_vis)/urdf/barrett_hand.xacro" />
 </robot>

File: ws_AF/src/baxter_common/robotiq_2f_85_gripper_vis/urdf/robotiq_arg2f.xacro (robot description, xacro)
@@ -33,5 +33,5 @@
   </xacro:macro>
   <!-- Electric Gripper Tip joint -->
-  <joint name="left_endpoint" type="fixed">
+  <joint name="left_endpoint_joint" type="fixed">
     <origin rpy="0 0 0" xyz="0 0 ${0.130324+0.02}"/> <!-- Value added from all z values manually-->
     <parent link="left_gripper_base"/>

File: ws_AF/src/baxter_common/robotiq_2f_85_gripper_vis/urdf/robotiq_arg2f_85_model_macro.xacro (robot description, xacro)
@@ -137,5 +137,5 @@
       <axis xyz="1 0 0" />
       <limit lower="0" upper="0.8757" velocity="2.0" effort="1000" />
-      <mimic joint="${prefix}left_outer_knuckle_joint" multiplier="1" offset="0" />
+      <mimic joint="${prefix}finger_joint" multiplier="1" offset="0" />
     </joint>
   </xacro:macro>
@@ -147,5 +147,5 @@
       <axis xyz="1 0 0" />
       <limit lower="0" upper="0.8757" velocity="2.0" effort="1000" />
-      <mimic joint="${prefix}left_outer_knuckle_joint" multiplier="-1" offset="0" />
+      <mimic joint="${prefix}finger_joint" multiplier="-1" offset="0" />
     </joint>
   </xacro:macro>
@@ -160,6 +160,6 @@
   <!-- LOADS FROM THE OTHER FILE -->
   <xacro:include filename="$(find robotiq_2f_85_gripper_vis)/urdf/robotiq_arg2f.xacro" />
-  <xacro:macro name="left_outer_knuckle_joint" params="prefix">
-    <joint name="${prefix}left_outer_knuckle_joint" type="revolute">
+  <xacro:macro name="finger_joint" params="prefix">
+    <joint name="${prefix}finger_joint" type="revolute">
       <origin xyz="0 -0.0306011 0.054904" rpy="0 0 ${pi}"/>
       <parent link="left_gripper_base" /> <!-- changed with name change for base-->
@@ -177,15 +177,15 @@
       <axis xyz="1 0 0" />
       <limit lower="0" upper="0.81" velocity="2.0" effort="1000" />
-      <mimic joint="${prefix}left_outer_knuckle_joint" multiplier="1" offset="0" />
+      <mimic joint="${prefix}finger_joint" multiplier="1" offset="0" />
     </joint>
     <xacro:finger_joints prefix="${prefix}" fingerprefix="right" reflect="-1.0"/>
   </xacro:macro>
   <!-- Initialization of all joints and links -->
-  <xacro:macro name="left_gripper_base" params="prefix">
+  <xacro:macro name="left_robotiq_gripper" params="prefix">
     <xacro:robotiq_arg2f_base_link prefix="${prefix}"/>
     <xacro:finger_links prefix="${prefix}" fingerprefix="left" stroke="85"/>
     <xacro:finger_links prefix="${prefix}" fingerprefix="right" stroke="85"/>
+    <xacro:finger_joint prefix="${prefix}"/>
     <xacro:right_outer_knuckle_joint prefix="${prefix}"/>
-    <xacro:left_outer_knuckle_joint prefix="${prefix}"/>
     <xacro:robotiq_arg2f_transmission prefix="${prefix}"/>
   </xacro:macro>

File: ws_AF/src/baxter_common/robotiq_2f_85_gripper_vis/urdf/robotiq_arg2f_transmission.xacro (robot description, xacro)
@@ -4,8 +4,8 @@
     <transmission name="${prefix}finger_joint_trans">
       <type>transmission_interface/SimpleTransmission</type>
-      <joint name="${prefix}finger_joint">
+      <joint name="left_outer_knuckle_joint">
         <hardwareInterface>PositionJointInterface</hardwareInterface>
       </joint>
-      <actuator name="${prefix}finger_joint_motor">
+      <actuator name="left_outer_knuckle_joint">
         <mechanicalReduction>1</mechanicalReduction>
       </actuator>

File: ws_AF/src/moveit_robots/baxter_moveit_config/baxter_moveit_config/config/robotiq_gripper.srdf.xacro (robot description, xacro)
@@ -5,25 +5,67 @@
 -->
 <robot xmlns:xacro="http://www.ros.org/wiki/xacro" name="robotiq_gripper">
-    <xacro:macro name="robotiq_gripper" params="side"> <!-- fingerprefix is like side[0]-->
-    <!-- Disable collision between two specific links: link1 and link2 -->
-    <disable_collisions link1="left_gripper" link2="left_inner_finger_pad" reason="Never" />
-    <disable_collisions link1="left_gripper" link2="left_inner_finger" reason="Never" />
-    <disable_collisions link1="left_gripper" link2="left_inner_knuckle" reason="Never" />
-    <disable_collisions link1="left_gripper" link2="left_outer_finger" reason="Never" />
-    <disable_collisions link1="left_gripper" link2="left_outer_knuckle" reason="Never" />
-    <disable_collisions link1="left_gripper" link2="right_inner_finger_pad" reason="Never" />
-    <disable_collisions link1="left_gripper" link2="right_inner_finger" reason="Never" />
-    <disable_collisions link1="left_gripper" link2="right_inner_knuckle" reason="Never" />
-    <disable_collisions link1="left_gripper" link2="right_outer_finger" reason="Never" />
-    <disable_collisions link1="left_gripper" link2="right_outer_knuckle" reason="Never" />
-    <disable_collisions link1="left_gripper" link2="${side}_hand" reason="Never" />
-    <disable_collisions link1="left_gripper" link2="${side}_hand_accelerometer" reason="Never" />
-    <disable_collisions link1="left_gripper" link2="${side}_hand_camera" reason="Never" />
-    <disable_collisions link1="left_gripper" link2="${side}_hand_range" reason="Never" />
-    <disable_collisions link1="left_gripper" link2="${side}_lower_elbow" reason="Never" />
-    <disable_collisions link1="left_gripper" link2="${side}_lower_forearm" reason="Never" />
-    <disable_collisions link1="left_gripper" link2="${side}_upper_forearm" reason="Never" />
-    <disable_collisions link1="left_gripper" link2="${side}_upper_forearm_visual" reason="Never" />
-    <disable_collisions link1="left_gripper" link2="${side}_wrist" reason="Never" />
+    <!-- Macro for robotiq_gripper Gripper (Left) FOR NOW -->
+    <!-- NOT CURRENTLY BEING USED, MIGHT BE NEEDED?-->
+    <xacro:macro name="robotiq_arg2f_85_model_macro">
+    <xacro:property name="gripper_side" value="l" scope="local"/> <!-- "l" is for left side -->
+    <!-- robotiq_arg2f_base_link -->
+    <disable_collisions link1="robotiq_arg2f_base_link" link2="${gripper_side}_gripper_l_finger" reason="Adjacent" />
+    <disable_collisions link1="robotiq_arg2f_base_link" link2="${gripper_side}_gripper_l_finger_tip" reason="Never" />
+    <disable_collisions link1="${side}_gripper_base" link2="${gripper_side}_gripper_r_finger" reason="Adjacent" />
+    <disable_collisions link1="${side}_gripper_base" link2="${gripper_side}_gripper_r_finger_tip" reason="Never" />
+    <!--  -->
+    <disable_collisions link1="${side}_gripper" link2="${gripper_side}_gripper_l_finger" reason="Default" />
+    <disable_collisions link1="${side}_gripper" link2="${gripper_side}_gripper_l_finger_tip" reason="Never" />
+    <disable_collisions link1="${side}_gripper" link2="${gripper_side}_gripper_r_finger" reason="Default" />
+    <disable_collisions link1="${side}_gripper" link2="${gripper_side}_gripper_r_finger_tip" reason="Never" />
+    <!--  -->
+    <disable_collisions link1="${gripper_side}_gripper_l_finger" link2="${gripper_side}_gripper_l_finger_tip" reason="Adjacent" />
+    <disable_collisions link1="${gripper_side}_gripper_l_finger" link2="${gripper_side}_gripper_r_finger" reason="Never" />
+    <disable_collisions link1="${gripper_side}_gripper_l_finger" link2="${gripper_side}_gripper_r_finger_tip" reason="Never" />
+    <disable_collisions link1="${gripper_side}_gripper_l_finger" link2="${side}_hand" reason="Never" />
+    <disable_collisions link1="${gripper_side}_gripper_l_finger" link2="${side}_hand_accelerometer" reason="Never" />
+    <disable_collisions link1="${gripper_side}_gripper_l_finger" link2="${side}_hand_camera" reason="Never" />
+    <disable_collisions link1="${gripper_side}_gripper_l_finger" link2="${side}_hand_range" reason="Never" />
+    <disable_collisions link1="${gripper_side}_gripper_l_finger" link2="${side}_lower_elbow" reason="Never" />
+    <disable_collisions link1="${gripper_side}_gripper_l_finger" link2="${side}_lower_forearm" reason="Never" />
+    <disable_collisions link1="${gripper_side}_gripper_l_finger" link2="${side}_upper_forearm" reason="Never" />
+    <disable_collisions link1="${gripper_side}_gripper_l_finger" link2="${side}_upper_forearm_visual" reason="Never" />
+    <disable_collisions link1="${gripper_side}_gripper_l_finger" link2="${side}_wrist" reason="Never" />
+    <disable_collisions link1="${gripper_side}_gripper_l_finger_tip" link2="${gripper_side}_gripper_r_finger" reason="Never" />
+    <disable_collisions link1="${gripper_side}_gripper_l_finger_tip" link2="${side}_hand" reason="Never" />
+    <disable_collisions link1="${gripper_side}_gripper_l_finger_tip" link2="${side}_hand_accelerometer" reason="Never" />
+    <disable_collisions link1="${gripper_side}_gripper_l_finger_tip" link2="${side}_hand_camera" reason="Never" />
+    <disable_collisions link1="${gripper_side}_gripper_l_finger_tip" link2="${side}_hand_range" reason="Never" />
+    <disable_collisions link1="${gripper_side}_gripper_l_finger_tip" link2="${side}_lower_elbow" reason="Never" />
+    <disable_collisions link1="${gripper_side}_gripper_l_finger_tip" link2="${side}_lower_forearm" reason="Never" />
+    <disable_collisions link1="${gripper_side}_gripper_l_finger_tip" link2="${side}_upper_elbow_visual" reason="Never" />
+    <disable_collisions link1="${gripper_side}_gripper_l_finger_tip" link2="${side}_upper_forearm" reason="Never" />
+    <disable_collisions link1="${gripper_side}_gripper_l_finger_tip" link2="${side}_upper_forearm_visual" reason="Never" />
+    <disable_collisions link1="${gripper_side}_gripper_l_finger_tip" link2="${side}_wrist" reason="Never" />
+    <!--  -->
+    <disable_collisions link1="${gripper_side}_gripper_r_finger" link2="${gripper_side}_gripper_r_finger_tip" reason="Adjacent" />
+    <disable_collisions link1="${gripper_side}_gripper_r_finger" link2="${side}_hand" reason="Never" />
+    <disable_collisions link1="${gripper_side}_gripper_r_finger" link2="${side}_hand_accelerometer" reason="Never" />
+    <disable_collisions link1="${gripper_side}_gripper_r_finger" link2="${side}_hand_camera" reason="Never" />
+    <disable_collisions link1="${gripper_side}_gripper_r_finger" link2="${side}_hand_range" reason="Never" />
+    <disable_collisions link1="${gripper_side}_gripper_r_finger" link2="${side}_lower_elbow" reason="Never" />
+    <disable_collisions link1="${gripper_side}_gripper_r_finger" link2="${side}_lower_forearm" reason="Never" />
+    <disable_collisions link1="${gripper_side}_gripper_r_finger" link2="${side}_upper_forearm" reason="Never" />
+    <disable_collisions link1="${gripper_side}_gripper_r_finger" link2="${side}_upper_forearm_visual" reason="Never" />
+    <disable_collisions link1="${gripper_side}_gripper_r_finger" link2="${side}_wrist" reason="Never" />
+    <disable_collisions link1="${gripper_side}_gripper_r_finger_tip" link2="${side}_hand" reason="Never" />
+    <disable_collisions link1="${gripper_side}_gripper_r_finger_tip" link2="${side}_hand_accelerometer" reason="Never" />
+    <disable_collisions link1="${gripper_side}_gripper_r_finger_tip" link2="${side}_hand_camera" reason="Never" />
+    <disable_collisions link1="${gripper_side}_gripper_r_finger_tip" link2="${side}_hand_range" reason="Never" />
+    <disable_collisions link1="${gripper_side}_gripper_r_finger_tip" link2="${side}_lower_elbow" reason="Never" />
+    <disable_collisions link1="${gripper_side}_gripper_r_finger_tip" link2="${side}_lower_forearm" reason="Never" />
+    <disable_collisions link1="${gripper_side}_gripper_r_finger_tip" link2="${side}_upper_elbow_visual" reason="Never" />
+    <disable_collisions link1="${gripper_side}_gripper_r_finger_tip" link2="${side}_upper_forearm" reason="Never" />
+    <disable_collisions link1="${gripper_side}_gripper_r_finger_tip" link2="${side}_upper_forearm_visual" reason="Never" />
+    <disable_collisions link1="${gripper_side}_gripper_r_finger_tip" link2="${side}_wrist" reason="Never" />
+    <!--  -->
+    <disable_collisions link1="${gripper_side}_gripper_l_finger_tip" link2="${gripper_side}_gripper_r_finger_tip" reason="Never" />
+    <disable_collisions link1="${gripper_side}_gripper_l_finger" link2="${gripper_side}_gripper_l_finger_tip" reason="Never" />
+    <disable_collisions link1="${gripper_side}_gripper_r_finger" link2="${gripper_side}_gripper_r_finger_tip" reason="Never" />
     </xacro:macro>
 </robot>
