Commit message: Got both in moveit Still neds work

File: ws_AF/src/baxter_common/baxter_description/urdf/left_end_effector.urdf.xacro (robot description, xacro)
@@ -1,7 +1,4 @@
 <?xml version="1.0" ?>
 <robot name="left_end_effector" xmlns:xacro="http://www.ros.org/wiki/xacro">
-  <!-- Define necessary properties for the gripper -->
-  <xacro:property name="dist_joint_multiplier" value="0.3" />
-  <xacro:property name="dist_joint_offset" value="0.75" />
   <!-- Include the Robotiq 2F-85 gripper Xacro file -->
   <xacro:include filename="$(find robotiq_2f_85_gripper_vis)/urdf/robotiq_arg2f_85_model_macro.xacro" />

File: ws_AF/src/baxter_common/baxter_description/urdf/right_end_effector.urdf.xacro (robot description, xacro)
@@ -1,10 +1,10 @@
 <?xml version="1.0" ?>
 <robot name="right_end_effector" xmlns:xacro="http://www.ros.org/wiki/xacro">
-  <!-- <xacro:include filename="$(find barrett_hand_vis)/urdf/bh282.urdf.xacro" />
+  <xacro:include filename="$(find barrett_hand_vis)/urdf/bh282.urdf.xacro" />
   <xacro:bhand_macro name="bh" parent="right_hand">
-    <origin xyz="0 0 0.5" rpy="0 0 0" />
-  </xacro:bhand_macro> -->
+    <origin xyz="0 0 0" rpy="0 0 1.5708" />
+  </xacro:bhand_macro>
   <!-- Import Rviz colors -->
-  <xacro:include filename="$(find barrett_hand_vis)/urdf/materials.xacro" />
+  <!-- <xacro:include filename="$(find barrett_hand_vis)/urdf/materials.xacro" />
   <joint name="base_joint" type="fixed">
     <origin xyz="0 0 0.002" rpy="0 0 4.7124"/>
@@ -12,4 +12,4 @@
     <child link="barrett_base_link"/>
   </joint>
-  <xacro:include filename="$(find barrett_hand_vis)/urdf/barrett_hand.xacro" />
+  <xacro:include filename="$(find barrett_hand_vis)/urdf/barrett_hand.xacro" /> -->
 </robot>
