Commit message: Everything is working

File: ws_AF/src/baxter_common/barrett_hand_vis/urdf/bh282.urdf.xacro (robot description, xacro)
@@ -54,5 +54,5 @@
 			  <mesh filename="package://barrett_hand_vis/meshes/knuckle_fixed.dae" />
 		   </geometry>
-		   <material name="Black"/>
+		   <color rgba="0.0 0.0 0.0 1.0"/>
 		 </visual>
 		 <collision>
@@ -83,5 +83,5 @@
 				  <mesh filename="package://barrett_hand_vis/meshes/finger.dae" />
 				</geometry>
-				<material name="Blue" />
+				<color rgba="0.0 0.0 0.8 1.0"/>
 			 </visual>
 			 <collision>
@@ -126,5 +126,5 @@
 			  <mesh filename="package://barrett_hand_vis/meshes/finger_tip.dae" />
 			</geometry>
-			<material name="Blue" />
+			<color rgba="0.0 0.0 0.8 1.0"/>
 		 </visual>
 		 <collision>
@@ -170,5 +170,5 @@
 				 <mesh filename="package://barrett_hand_vis/meshes/knuckle.dae" />
 			  </geometry>
-			  <material name="Green" />
+			  <color rgba="0.0 0.8 0.0 1.0"/>
 			</visual>
 			<collision>
@@ -211,5 +211,5 @@
 				  <mesh filename="package://barrett_hand_vis/meshes/finger.dae" />
 				</geometry>
-				<material name="Blue" />
+				<color rgba="0.0 0.0 0.8 1.0"/>
 			 </visual>
 			 <collision>
@@ -254,5 +254,5 @@
 			  <mesh filename="package://barrett_hand_vis/meshes/finger_tip.dae" />
 			</geometry>
-			<material name="Blue" />
+			<color rgba="0.0 0.0 0.8 1.0"/>
 		 </visual>
 		 <collision>
@@ -298,5 +298,5 @@
 				 <mesh filename="package://barrett_hand_vis/meshes/knuckle.dae" />
 			  </geometry>
-			  <material name="Green" />
+			  <color rgba="0.0 0.8 0.0 1.0"/>
 			</visual>
 			<collision>
@@ -340,5 +340,5 @@
 				  <mesh filename="package://barrett_hand_vis/meshes/finger.dae" />
 				</geometry>
-				<material name="Blue" />
+				<color rgba="0.0 0.0 0.8 1.0"/>
 			 </visual>
 			 <collision>
@@ -383,5 +383,5 @@
 			  <mesh filename="package://barrett_hand_vis/meshes/finger_tip.dae" />
 			</geometry>
-			<material name="Blue" />
+			<color rgba="0.0 0.0 0.8 1.0"/>
 		 </visual>
 		 <collision>

File: ws_AF/src/baxter_common/baxter_description/urdf/baxter.urdf (robot description, URDF)
Before this commit: robot baxter, 67 links, 66 joints
Links:
- removed link barrett_base_link
- removed link finger_1_dist_link
- removed link finger_1_med_link
- removed link finger_1_prox_link
- removed link finger_2_dist_link
- removed link finger_2_med_link
- removed link finger_2_prox_link
- removed link finger_3_dist_link
- removed link finger_3_med_link
- removed link palm_frame
- added link bh_base_link, mass 3.0; collision mesh filename=package://barrett_hand_vis/meshes/palm_282.dae; visual mesh filename=package://barrett_hand_vis/meshes/palm_282.dae
- added link bh_finger_11_link, mass 0.1; collision mesh filename=package://barrett_hand_vis/meshes/knuckle.dae; visual mesh filename=package://barrett_hand_vis/meshes/knuckle.dae
- added link bh_finger_12_link, mass 0.1; collision mesh filename=package://barrett_hand_vis/meshes/finger.dae; visual mesh filename=package://barrett_hand_vis/meshes/finger.dae
- added link bh_finger_13_link, mass 0.1; collision mesh filename=package://barrett_hand_vis/meshes/finger_tip.dae; visual mesh filename=package://barrett_hand_vis/meshes/finger_tip.dae
- added link bh_finger_21_link, mass 0.1; collision mesh filename=package://barrett_hand_vis/meshes/knuckle.dae; visual mesh filename=package://barrett_hand_vis/meshes/knuckle.dae
- added link bh_finger_22_link, mass 0.1; collision mesh filename=package://barrett_hand_vis/meshes/finger.dae; visual mesh filename=package://barrett_hand_vis/meshes/finger.dae
- added link bh_finger_23_link, mass 0.1; collision mesh filename=package://barrett_hand_vis/meshes/finger_tip.dae; visual mesh filename=package://barrett_hand_vis/meshes/finger_tip.dae
- added link bh_finger_31_link, mass 0.1; collision mesh filename=package://barrett_hand_vis/meshes/knuckle_fixed.dae; visual mesh filename=package://barrett_hand_vis/meshes/knuckle_fixed.dae
- added link bh_finger_32_link, mass 0.1; collision mesh filename=package://barrett_hand_vis/meshes/finger.dae; visual mesh filename=package://barrett_hand_vis/meshes/finger.dae
- added link bh_finger_33_link, mass 0.1; collision mesh filename=package://barrett_hand_vis/meshes/finger_tip.dae; visual mesh filename=package://barrett_hand_vis/meshes/finger_tip.dae
Joints:
- removed joint base_joint
- removed joint finger_1_dist_joint
- removed joint finger_1_med_joint
- removed joint finger_1_prox_joint
- removed joint finger_2_dist_joint
- removed joint finger_2_med_joint
- removed joint finger_2_prox_joint
- removed joint finger_3_dist_joint
- removed joint finger_3_med_joint
- removed joint palm_joint
- added joint bh_base_joint: type fixed, parent right_hand, child bh_base_link, origin xyz=0 0 0 rpy=0 0 1.5708
- added joint bh_j11_joint: type revolute, parent bh_base_link, child bh_finger_11_link, origin xyz=-0.025 0 0.0252 rpy=0 0 1.5708, axis 0 0 -1, limit lower=0 upper=3.1416 effort=30.0 velocity=2.0
- added joint bh_j12_joint: type revolute, parent bh_finger_11_link, child bh_finger_12_link, origin xyz=-0.05 0 0.0339 rpy=1.5708 0 0, axis 0 0 -1, limit lower=0.0 upper=2.44 effort=30.0 velocity=2.0
- added joint bh_j13_joint: type revolute, parent bh_finger_12_link, child bh_finger_13_link, origin xyz=-0.069936 0.003 0 rpy=0 0 0, axis 0 0 -1, limit lower=0.0 upper=0.84 effort=30.0 velocity=2.0, mimic joint=bh_j12_joint multiplier=0.3442622950819672
- added joint bh_j21_joint: type revolute, parent bh_base_link, child bh_finger_21_link, origin xyz=0.025 0 0.0252 rpy=0 0 1.5708, axis 0 0 1, limit lower=0 upper=3.1416 effort=30.0 velocity=2.0, mimic joint=bh_j11_joint multiplier=1
- added joint bh_j22_joint: type revolute, parent bh_finger_21_link, child bh_finger_22_link, origin xyz=-0.05 0 0.0339 rpy=1.5708 -8.8281E-17 0, axis 0 0 -1, limit lower=0.0 upper=2.44 effort=30.0 velocity=2.0
- added joint bh_j23_joint: type revolute, parent bh_finger_22_link, child bh_finger_23_link, origin xyz=-0.069936 0.003 0 rpy=0 0 0, axis 0 0 -1, limit lower=0.0 upper=0.84 effort=30.0 velocity=2.0, mimic joint=bh_j22_joint multiplier=0.3442622950819672
- added joint bh_j31_joint: type fixed, parent bh_base_link, child bh_finger_31_link, origin xyz=0 0 0.0252 rpy=0 0 -1.570796327
- added joint bh_j32_joint: type revolute, parent bh_finger_31_link, child bh_finger_32_link, origin xyz=-0.05 0 0.0339 rpy=1.5708 -8.8281E-17 0, axis 0 0 -1, limit lower=0.0 upper=2.44 effort=30.0 velocity=2.0
- added joint bh_j33_joint: type revolute, parent bh_finger_32_link, child bh_finger_33_link, origin xyz=-0.069936 0.003 0 rpy=0 0 0, axis 0 0 -1, limit lower=0.0 upper=0.84 effort=30.0 velocity=2.0, mimic joint=bh_j32_joint multiplier=0.3442622950819672

File: ws_AF/src/baxter_common/baxter_description/urdf/right_end_effector.urdf.xacro (robot description, xacro)
@@ -2,4 +2,5 @@
 <robot name="right_end_effector" xmlns:xacro="http://www.ros.org/wiki/xacro">
   <xacro:include filename="$(find barrett_hand_vis)/urdf/bh282.urdf.xacro" />
+  <xacro:include filename="$(find barrett_hand_vis)/urdf/materials.xacro" />
   <xacro:bhand_macro name="bh" parent="right_hand">
     <origin xyz="0 0 0" rpy="0 0 1.5708" />

File: ws_AF/src/baxter_common/robotiq_2f_85_gripper_vis/urdf/robotiq_arg2f.xacro (robot description, xacro)
@@ -41,5 +41,5 @@
   <link name="left_gripper">
     <inertial>
-      <origin rpy="0 0 0" xyz="0 0 0"/>
+      <origin rpy="0 0 1" xyz="0 0 0"/>
       <mass value="0.0001"/>
       <inertia ixx="0" ixy="0" ixz="0" iyy="0" iyz="0" izz="0.0"/>
